Commit message: fix(adam-sp): refine self-collision geometry

File: source/instinctlab/instinctlab/assets/resources/adam_sp/urdf/adam_sp_23_dof.urdf (robot description, URDF)
Before this commit: robot adam_sp, 55 links, 54 joints
Links:
- link left_hip_roll_link: geometry collision cylinder length=0.08 radius=0.05; collision sphere radius=0.05
- link right_hip_roll_link: geometry collision cylinder length=0.08 radius=0.05; collision sphere radius=0.05
